File: hardware/trippy_shadows/trippy_shadows.kicad_pcb (KiCad board)
At the start: 2 copper layers, 71 x 48 mm, 34 parts, among them J1 ISP, J10 JST conn, J2 GPIO, J3 DEBUG, J4 PWR, J5 JST conn, J6 JST conn, J7 JST conn, J8 JST conn, J9 JST conn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

Commit message: Commit latest board design
Parts:
- removed J2: GPIO, Connector_PinHeader_2.54mm:PinHeader_2x04_P2.54mm_Vertical
- added R10: 10k, Resistor_SMD:R_0805_2012Metric, F.Cu at (161.1, 78.5)
- added R11: 10k, Resistor_SMD:R_0805_2012Metric, F.Cu at (161.2, 92.8)
- added R12: 10k, Resistor_SMD:R_0805_2012Metric, F.Cu at (151.2, 93.0)
- added R13: 10k, Resistor_SMD:R_0805_2012Metric, F.Cu at (142.0, 84.0)
- added R8: 10k, Resistor_SMD:R_0805_2012Metric, F.Cu at (141.1, 78.3)
- added R9: 10k, Resistor_SMD:R_0805_2012Metric, F.Cu at (151.2, 78.5)
- added RV1: 10k, Potentiometer_THT:Potentiometer_Alps_RK09K_Single_Vertical, F.Cu at (125.8, 66.0)
- J10, J5, J6, J7, J8, J9: value JST conn -> S2B-PH-KL(LF)(SN); footprint Connector_JST:JST_PH_B2B-PH-K_1x02_P2.00mm_Vertical -> Connector_JST:JST_PH_S2B-PH-K_1x02_P2.00mm_Horizontal
- J3: value DEBUG -> Debug; footprint Connector_PinHeader_2.54mm:PinHeader_2x03_P2.54mm_Vertical -> Connector_PinHeader_2.54mm:PinHeader_1x03_P2.54mm_Vertical
- J4: value PWR -> JST_PH_B2B-PH-K; footprint TerminalBlock:TerminalBlock_bornier-2_P5.08mm -> Connector_JST:JST_PH_B2B-PH-K_1x02_P2.00mm_Vertical
- R2, R3, R4, R5, R6, R7: value R -> 2.7k
- moved J4 47.3 mm to (144.9, 65.6), turned to 0 degrees
- moved J3 35.8 mm to (125.6, 101.0)
- moved J1 29.5 mm to (130.5, 94.2)
- moved C8 23.1 mm to (131.0, 76.5), turned to 180 degrees
- moved C1 18.5 mm to (131.0, 90.8), turned to 0 degrees
- moved R1 15.7 mm to (125.3, 78.4), turned to 90 degrees
- moved U1 8.75 mm to (131.8, 84.1), turned to -90 degrees
- moved C6 4.96 mm to (149.0, 84.0)
- moved J7 2.93 mm to (173.6, 95.9), turned to 90 degrees
- moved J8 2.64 mm to (147.6, 103.5)
- moved J6 2.17 mm to (173.4, 86.1), turned to 90 degrees
- moved J10 1.10 mm to (168.0, 103.5)
- moved J5 1.03 mm to (173.3, 75.8), turned to 90 degrees
- moved J9 0.92 mm to (157.8, 103.5)
Connections:
- J3 pad 1: /RXD -> GND
- J3 pad 2: /SDA -> /RXD
- U1 pad 1: /DRV4 -> /DRV1
- U1 pad 10: /GPIO5 -> unconnected-(U1-PD6-Pad10)
- U1 pad 11: /GPIO6 -> unconnected-(U1-PD7-Pad11)
- U1 pad 12: /GPIO0 -> unconnected-(U1-PB0-Pad12)
- U1 pad 13: /GPIO1 -> unconnected-(U1-PB1-Pad13)
- U1 pad 14: /GPIO2 -> unconnected-(U1-PB2-Pad14)
- U1 pad 2: /DRV5 -> /DRV0
- U1 pad 20: unconnected-(U1-AREF-Pad20) -> VCC
- U1 pad 22: unconnected-(U1-ADC7-Pad22) -> Net-(U1-ADC7)
- U1 pad 23: /DRV0 -> /DRV3
- U1 pad 24: /DRV1 -> /DRV4
- U1 pad 25: /DRV2 -> /DRV5
- U1 pad 26: /DRV3 -> /DRV2
- U1 pad 27: /SDA -> unconnected-(U1-PC4-Pad27)
- U1 pad 28: /SCL -> unconnected-(U1-PC5-Pad28)
- U1 pad 32: /INT0 -> unconnected-(U1-PD2-Pad32)
- U1 pad 7: /GPIO3 -> unconnected-(U1-XTAL1/PB6-Pad7)
- U1 pad 8: /GPIO4 -> unconnected-(U1-XTAL2/PB7-Pad8)
Routing:
- net /GPIO6: track 38.7 -> 0.00 mm, vias 3 -> 0
- net /GPIO2: track 38.0 -> 0.00 mm, vias 3 -> 0
- net /INT0: track 37.8 -> 0.00 mm, vias 2 -> 0
- net /GPIO1: track 31.8 -> 0.00 mm, vias 3 -> 0
- net /GPIO4: track 26.4 -> 0.00 mm
- net Net-(U1-ADC7): track 0.00 -> 26.1 mm, vias 0 -> 1
- net /GPIO5: track 25.9 -> 0.00 mm, vias 3 -> 0
- net /GPIO0: track 25.0 -> 0.00 mm, vias 2 -> 0
- net /SCL: track 24.5 -> 0.00 mm, vias 1 -> 0
- net /SDA: track 22.2 -> 0.00 mm
- net //RES: track 45.0 -> 25.6 mm, vias 1 -> 2
- net /DRV2: track 53.4 -> 35.1 mm
- net /GPIO3: track 17.9 -> 0.00 mm
- net /DRV4: track 36.0 -> 21.2 mm
- net /DRV5: track 44.9 -> 30.4 mm
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Other:
- board size 71 x 48 mm -> 55.8 x 48 mm
- board text added: "+"
- board text added: "-"
- board text added: "2.7k"
- board text added: "Diablo's Bouqet (c) Mayhem Chaos 2025-01-05"
- board text added: "Diablo's Bouqet 2025-01-05"
- board text added: "LED0"
- board text added: "LED1"
- board text added: "LED2"
- board text added: "LED3"
- board text added: "LED4"
- board text added: "LED5"
- board text added: "PWR"
- board text added: "RXD"
- board text added: "TXD"
- board text removed: "GP0"
- board text removed: "GP1"
- board text removed: "GP2"
- board text removed: "GP3"
- board text removed: "GP4"
- board text removed: "GP5"
- board text removed: "GP6"
- board text removed: "INT0"
- board text removed: "RX"
- board text removed: "Radj"
- board text removed: "SCL"
- board text removed: "SDA"
- board text removed: "TX"
- board text removed: "Trippy Shadows 6-way LED driver (c) Mayhem Chaos 2024-12-23"

Commit message: Updated schematic to move to working adc
Connections:
- RV1 pad 2: Net-(U1-ADC7) -> /POT
- U1 pad 22: Net-(U1-ADC7) -> unconnected-(U1-ADC7-Pad22)
- U1 pad 27: unconnected-(U1-PC4-Pad27) -> /POT
Routing:
- net Net-(U1-ADC7): track 26.1 -> 0.00 mm, vias 1 -> 0
- net /POT: track 0.00 -> 26.0 mm, vias 0 -> 1
Other:
- board text added: "Diablo's Bouquet (c) Mayhem Chaos 2025-01-15"
- board text added: "Diablo's Bouquet 2025-01-15"
- board text removed: "Diablo's Bouqet 2025-01-05"
Changed lines of the file:
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@@
 	(net 5 "/{slash}RES")
 	(net 6 "/MOSI")
-	(net 7 "Net-(U1-ADC7)")
+	(net 7 "/POT")
 	(net 8 "unconnected-(U1-PB0-Pad12)")
 	(net 9 "unconnected-(U1-PD2-Pad32)")
 	(net 10 "unconnected-(U1-XTAL2{slash}PB7-Pad8)")
-	(net 11 "unconnected-(U1-PC4-Pad27)")
+	(net 11 "unconnected-(U1-ADC7-Pad22)")
 	(net 12 "unconnected-(U1-PB2-Pad14)")
 	(net 13 "unconnected-(U1-PD7-Pad11)")
@@
 		(tags "capacitor")
 		(property "Reference" "C1"
-			(at 0 -1.68 360)
+			(at 0 -1.68 0)
 			(layer "F.SilkS")
 			(hide yes)
@@
 		)
 		(property "Value" "100nF"
-			(at -13.4 -13.15 360)
+			(at -13.4 -13.15 0)
 			(layer "F.SilkS")
 			(hide yes)
@@
 			(size 1.6 0.55)
 			(layers "F.Cu" "F.Paste" "F.Mask")
-			(net 7 "Net-(U1-ADC7)")
+			(net 11 "unconnected-(U1-ADC7-Pad22)")
 			(pinfunction "ADC7")
-			(pintype "input")
+			(pintype "input+no_connect")
 		)
 		(pad "23" smd rect
@@
 			(size 1.6 0.55)
 			(layers "F.Cu" "F.Paste" "F.Mask")
-			(net 11 "unconnected-(U1-PC4-Pad27)")
+			(net 7 "/POT")
 			(pinfunction "PC4")
-			(pintype "bidirectional+no_connect")
+			(pintype "bidirectional")
 		)
 		(pad "28" smd rect
@@
 		(tags "capacitor")
 		(property "Reference" "C6"
-			(at 0 -1.68 360)
+			(at 0 -1.68 0)
 			(layer "F.SilkS")
 			(hide yes)
@@
 		)
 		(property "Value" "100nF"
-			(at -2.45 1.4 360)
+			(at -2.45 1.4 0)
 			(layer "F.SilkS")
 			(hide yes)
@@
 		(tags "capacitor")
 		(property "Reference" "C8"
-			(at 0 -1.68 360)
+			(at 0 -1.68 0)
 			(layer "F.SilkS")
 			(hide yes)
@@
 		)
 		(property "Value" "100nF"
-			(at 3 1.75 360)
+			(at 3 1.75 0)
 			(layer "F.SilkS")
 			(effects
@@
 			(layers "*.Cu" "*.Mask")
 			(remove_unused_layers no)
-			(net 7 "Net-(U1-ADC7)")
+			(net 7 "/POT")
 			(pinfunction "2")
 			(pintype "passive")
@@
 		)
 	)
-	(gr_text "Diablo's Bouqet 2025-01-05"
+	(gr_text "Diablo's Bouquet 2025-01-15"
 		(at 124.025 108.075 0)
 		(layer "F.SilkS")
@@
 		)
 	)
-	(gr_text "Diablo's Bouqet\n(c) Mayhem Chaos\n2025-01-05"
+	(gr_text "Diablo's Bouquet\n(c) Mayhem Chaos\n2025-01-15"
 		(at 151.125 68.2 0)
 		(layer "F.SilkS")
@@
 	)
 	(segment
-		(start 132.95 88.35)
-		(end 132.95 85.9)
-		(width 0.2)
-		(layer "F.Cu")
-		(net 7)
-	)
-	(segment
-		(start 132.95 85.9)
-		(end 132.65 85.6)
+		(start 130.55 82.65)
+		(end 130.55 84.8)
 		(width 0.2)
 		(layer "F.Cu")
@@
 	)
 	(segment
-		(start 130.55 85.6)
-		(end 130.55 82.65)
+		(start 131.05 85.3)
+		(end 136 85.3)
 		(width 0.2)
 		(layer "F.Cu")
@@
 	)
 	(segment
-		(start 132.65 85.6)
-		(end 130.55 85.6)
+		(start 130.55 84.8)
+		(end 131.05 85.3)
 		(width 0.2)
 		(layer "F.Cu")
